File: Hardware/Qwiic Environmental BME680.brd (EAGLE design)
At the start: 25.4 x 25.4 mm, 54 parts, among them J2 SPI, J5 QWIIC, J7 QWIIC, U1 BME680BME680

Commit message: adding buzzard for address
Parts:
- added U$33: (no value), buzzard_labels:ADR#_0X770
Changed lines of the file:
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@@
 <?xml version="1.0" encoding="utf-8"?>
 <!DOCTYPE eagle SYSTEM "eagle.dtd">
-<eagle version="9.5.2">
+<eagle version="9.6.0">
 <drawing>
 <settings>
@@
 <element name="FD2" library="SparkFun-Aesthetics" package="FIDUCIAL-MICRO" value="FIDUCIALUFIDUCIAL" x="24.13" y="20.32" smashed="yes" rot="MR0"/>
 <element name="FD4" library="SparkFun-Aesthetics" package="FIDUCIAL-MICRO" value="FIDUCIALUFIDUCIAL" x="1.27" y="1.27" smashed="yes"/>
+<element name="U$33" library="buzzard_labels" package="ADR#_0X770" value="" x="17.145" y="9.398" smashed="yes" rot="MR0"/>
 </elements>
 <signals>

Commit message: pre design review changes
Parts:
- removed U$31: (no value), SparkFun-Aesthetics:SFE_LOGO_FLAME_.3
- added D1: RED, SparkFun-LED:LED-0603
- added LOGO2: SFE_LOGO_NAME_FLAME.1_INCH, SparkFun-Aesthetics:SFE_LOGO_NAME_FLAME_.1
- added PWRLED: JUMPER-SMT_2_NC_TRACE_SILK, SparkFun-Jumpers:SMT-JUMPER_2_NC_TRACE_SILK
- added R2: 1k, SparkFun-Resistors:0603
- added U$34: (no value), SparkFun-Buzzard:PWR_TO
- R1, R3, R4, R5: device SparkFun-Resistors:0603 -> SparkFun-Resistors:0603@1
- U$32: device SparkFun-Aesthetics:SFE_LOGO_NAME_FLAME_.1 -> SparkFun-Aesthetics:QWIIC_5MM
- U1: value BME680BME680 -> BME680
- moved U$32 11.2 mm to (22.2, 17.4), flipped to the top
- moved LOGO1 2.74 mm to (20.3, 1.52)
Connections:
- new net N$1: PWRLED.1, R2.2
- new net N$3: D1.A, R2.1
- net 3.3V: now also PWRLED.2
- net GND: now also D1.C
Routing:
- net 3.3V: track 51.7 -> 64.4 mm, vias 4 -> 5
- net SCK/SCL: track 53.6 -> 49.5 mm, vias 1 -> 2
- net N$1: track 0.00 -> 1.99 mm
- net N$3: track 0.00 -> 1.66 mm
Other:
- board text added: "Units in Inches"

Commit message: post checklist/review changes
Parts:
- added LOGO4: SFE_LOGO_FLAME.1_INCH, SparkFun-Aesthetics:SFE_LOGO_FLAME_.1
- J1: value (none) -> I2C
- U1: value BME680 -> BME680 Air Quality Sensor
- moved U$13 4.83 mm to (8.89, 6.35), turned to 270 degrees
- moved U$14 4.83 mm to (8.89, 1.52), turned to 90 degrees
Routing:
- net 3.3V: track 64.4 -> 69.3 mm, vias 5 -> 6
- net SCK/SCL: track 49.5 -> 50.3 mm
