File: Hardware/Qwiic Environmental BME680.sch (EAGLE design)
At the start: 22 parts, among them J2 SPI, J5 QWIIC, J7 QWIIC, U1 BME680BME680

Commit message: pre design review changes
Parts:
- added D1: RED, SparkFun-LED:LED-RED0603
- added LOGO2: SFE_LOGO_NAME_FLAME.1_INCH, SparkFun-Aesthetics:SFE_LOGO_NAME_FLAME.1_INCH
- added PWRLED: JUMPER-SMT_2_NC_TRACE_SILK, SparkFun-Jumpers:JUMPER-SMT_2_NC_TRACE_SILK
- added R2: 1k, SparkFun-Resistors:1KOHM-0603-1/10W-1%
- U1: value BME680BME680 -> BME680; device SparkFun-Sensors:BME680BME680 -> SparkFun-Sensors:BME680-LGA
Connections:
- new net N$1: PWRLED.1, R2.2
- new net N$3: D1.A, R2.1
- net 3.3V: now also PWRLED.2
- net GND: now also D1.C
Other:
- note added: "Clear the I2CPU Jumper to disconnect I2C Pull-up resistors"
- note added: "Cut the PWR jumper to disable the power LED"
- note added: "Must be open for SPI"
- note added: "Power"
- note added: "VDD: 1.71-3.6 V VDDIO: 1.2-3.6 V"
Changed lines of the file:
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@@
 <?xml version="1.0" encoding="utf-8"?>
 <!DOCTYPE eagle SYSTEM "eagle.dtd">
-<eagle version="9.5.2">
+<eagle version="9.6.0">
 <drawing>
 <settings>
@@
 <part name="LOGO1" library="SparkFun-Aesthetics" deviceset="OSHW-LOGO" device="MINI"/>
 <part name="R5" library="SparkFun-Resistors" deviceset="4.7KOHM" device="-0603-1/10W-1%" value="4.7k"/>
-<part name="U1" library="SparkFun-Sensors" deviceset="BME680" device="BME680"/>
+<part name="U1" library="SparkFun-Sensors" deviceset="BME680" device="-LGA" value="BME680"/>
 <part name="SUPPLY1" library="SparkFun-PowerSymbols" deviceset="3.3V" device=""/>
 <part name="J1" library="SparkFun-Connectors" deviceset="CONN_04" device="1X04_NO_SILK"/>
@@
 <part name="FD2" library="SparkFun-Aesthetics" deviceset="FIDUCIAL" device="UFIDUCIAL"/>
 <part name="FD4" library="SparkFun-Aesthetics" deviceset="FIDUCIAL" device="UFIDUCIAL"/>
+<part name="LOGO2" library="SparkFun-Aesthetics" deviceset="SFE_LOGO_NAME_FLAME" device=".1_INCH"/>
+<part name="R2" library="SparkFun-Resistors" deviceset="1KOHM" device="-0603-1/10W-1%" value="1k"/>
+<part name="SUPPLY6" library="SparkFun-PowerSymbols" deviceset="3.3V" device=""/>
+<part name="D1" library="SparkFun-LED" deviceset="LED-RED" device="0603" value="RED"/>
+<part name="GND1" library="SparkFun" deviceset="GND" device=""/>
+<part name="PWRLED" library="SparkFun-Jumpers" deviceset="JUMPER-SMT_2_NC_TRACE" device="_SILK" package3d_urn="urn:adsk.eagle:package:39281/1" value="JUMPER-SMT_2_NC_TRACE_SILK"/>
 </parts>
 <sheets>
@@
 <text x="2.54" y="96.52" size="2.54" layer="97" font="vector">Connections</text>
 <text x="169.672" y="7.366" size="2.54" layer="94" font="vector">A. England</text>
+<text x="2.54" y="175.26" size="1.778" layer="97" font="vector">VDD: 1.71-3.6 V
+VDDIO: 1.2-3.6 V</text>
+<text x="172.72" y="114.3" size="1.778" layer="97" font="vector">Must be open for SPI</text>
+<text x="152.4" y="162.56" size="1.778" layer="97" font="vector">Clear the I2CPU Jumper to disconnect
+I2C Pull-up resistors</text>
+<text x="41.148" y="124.206" size="1.778" layer="97" font="vector">Power</text>
+<text x="38.1" y="142.24" size="1.778" layer="97" font="vector">Cut the PWR
+jumper to disable
+the power LED</text>
 </plain>
 <instances>
@@
 <instance part="FD2" gate="G$1" x="238.76" y="20.32" smashed="yes"/>
 <instance part="FD4" gate="G$1" x="236.22" y="17.78" smashed="yes"/>
+<instance part="LOGO2" gate="G$1" x="190.5" y="38.1" smashed="yes"/>
+<instance part="R2" gate="G$1" x="35.56" y="137.16" smashed="yes" rot="R90">
+<attribute name="NAME" x="34.036" y="137.16" size="1.778" layer="95" font="vector" rot="R90" align="bottom-center"/>
+<attribute name="VALUE" x="37.084" y="137.16" size="1.778" layer="96" font="vector" rot="R90" align="top-center"/>
+</instance>
+<instance part="SUPPLY6" gate="G$1" x="35.56" y="157.48" smashed="yes">
+<attribute name="VALUE" x="35.56" y="160.274" size="1.778" layer="96" font="vector" align="bottom-center"/>
+</instance>
+<instance part="D1" gate="G$1" x="35.56" y="127" smashed="yes">
+<attribute name="NAME" x="32.131" y="122.428" size="1.778" layer="95" font="vector" rot="R90"/>
+<attribute name="VALUE" x="37.465" y="122.428" size="1.778" layer="96" font="vector" rot="R90" align="top-left"/>
+</instance>
+<instance part="GND1" gate="1" x="35.56" y="116.84" smashed="yes">
+<attribute name="VALUE" x="33.02" y="114.3" size="1.778" layer="96" font="vector"/>
+</instance>
+<instance part="PWRLED" gate="G$1" x="35.56" y="149.86" smashed="yes" rot="R90">
+<attribute name="NAME" x="38.1" y="149.86" size="1.778" layer="95" font="vector"/>
+</instance>
 </instances>
 <busses>
@@
 <pinref part="SUPPLY1" gate="G$1" pin="3.3V"/>
 </segment>
+<segment>
+<pinref part="SUPPLY6" gate="G$1" pin="3.3V"/>
+<pinref part="PWRLED" gate="G$1" pin="2"/>
+<wire x1="35.56" y1="157.48" x2="35.56" y2="154.94" width="0.1524" layer="91"/>
+</segment>
 </net>
 <net name="GND" class="0">
@@
 <wire x1="134.62" y1="48.26" x2="134.62" y2="45.72" width="0.1524" layer="91"/>
 <pinref part="GND11" gate="1" pin="GND"/>
+</segment>
+<segment>
+<pinref part="D1" gate="G$1" pin="C"/>
+<pinref part="GND1" gate="1" pin="GND"/>
+<wire x1="35.56" y1="119.38" x2="35.56" y2="121.92" width="0.1524" layer="91"/>
 </segment>
 </net>
@@
 </segment>
 </net>
+<net name="N$3" class="0">
+<segment>
+<pinref part="R2" gate="G$1" pin="1"/>
+<pinref part="D1" gate="G$1" pin="A"/>
+<wire x1="35.56" y1="129.54" x2="35.56" y2="132.08" width="0.1524" layer="91"/>
+</segment>
+</net>
+<net name="N$1" class="0">
+<segment>
+<pinref part="PWRLED" gate="G$1" pin="1"/>
+<pinref part="R2" gate="G$1" pin="2"/>
+<wire x1="35.56" y1="144.78" x2="35.56" y2="142.24" width="0.1524" layer="91"/>
+</segment>
+</net>
 </nets>
 </sheet>
@@
 </drawing>
 <compatibility>
+<note version="6.3" minversion="6.2.2" severity="warning">
+Since Version 6.2.2 text objects can contain more than one line,
+which will not be processed correctly with this version.
+</note>
 <note version="8.3" severity="warning">
 Since Version 8.3, EAGLE supports URNs for individual library

Commit message: post checklist/review changes
Parts:
- added LOGO4: SFE_LOGO_FLAME.1_INCH, SparkFun-Aesthetics:SFE_LOGO_FLAME.1_INCH
- J1: value (none) -> I2C
- U1: value BME680 -> BME680 Air Quality Sensor
Changed lines of the file:
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@@
 <part name="LOGO1" library="SparkFun-Aesthetics" deviceset="OSHW-LOGO" device="MINI"/>
 <part name="R5" library="SparkFun-Resistors" deviceset="4.7KOHM" device="-0603-1/10W-1%" value="4.7k"/>
-<part name="U1" library="SparkFun-Sensors" deviceset="BME680" device="-LGA" value="BME680"/>
+<part name="U1" library="SparkFun-Sensors" deviceset="BME680" device="-LGA" value="BME680 Air Quality Sensor"/>
 <part name="SUPPLY1" library="SparkFun-PowerSymbols" deviceset="3.3V" device=""/>
-<part name="J1" library="SparkFun-Connectors" deviceset="CONN_04" device="1X04_NO_SILK"/>
+<part name="J1" library="SparkFun-Connectors" deviceset="CONN_04" device="1X04_NO_SILK" value="I2C"/>
 <part name="LOGO3" library="SparkFun-Aesthetics" deviceset="REVISION" device=""/>
 <part name="FD2" library="SparkFun-Aesthetics" deviceset="FIDUCIAL" device="UFIDUCIAL"/>
@@
 <part name="GND1" library="SparkFun" deviceset="GND" device=""/>
 <part name="PWRLED" library="SparkFun-Jumpers" deviceset="JUMPER-SMT_2_NC_TRACE" device="_SILK" package3d_urn="urn:adsk.eagle:package:39281/1" value="JUMPER-SMT_2_NC_TRACE_SILK"/>
+<part name="LOGO4" library="SparkFun-Aesthetics" deviceset="SFE_LOGO_FLAME" device=".1_INCH"/>
 </parts>
 <sheets>
@@
 <attribute name="NAME" x="38.1" y="149.86" size="1.778" layer="95" font="vector"/>
 </instance>
+<instance part="LOGO4" gate="G$1" x="223.012" y="50.8" smashed="yes"/>
 </instances>
 <busses>
@@
 <net name="SDO/ADR" class="0">
 <segment>
-<wire x1="121.92" y1="132.08" x2="167.64" y2="132.08" width="0.1524" layer="91"/>
+<wire x1="121.92" y1="132.08" x2="129.54" y2="132.08" width="0.1524" layer="91"/>
 <pinref part="ADDR" gate="G$1" pin="2"/>
+<wire x1="129.54" y1="132.08" x2="167.64" y2="132.08" width="0.1524" layer="91"/>
 <wire x1="167.64" y1="132.08" x2="167.64" y2="129.54" width="0.1524" layer="91"/>
 <junction x="167.64" y="132.08"/>
@@
 <wire x1="167.64" y1="132.08" x2="167.64" y2="134.62" width="0.1524" layer="91"/>
 <pinref part="U1" gate="G$1" pin="SDO/ADR"/>
-</segment>
-<segment>
+<wire x1="129.54" y1="132.08" x2="129.54" y2="129.54" width="0.1524" layer="91"/>
+<junction x="129.54" y="132.08"/>
+<wire x1="129.54" y1="129.54" x2="132.08" y2="129.54" width="0.1524" layer="91"/>
+<label x="132.08" y="129.54" size="1.27" layer="95" font="vector" xref="yes"/>
+</segment>
+<segment>
